File: RC6802 CPU/RC6802 CPU.sch (KiCad schematic (older format))
At the start: 33 parts, among them J1 RC6802_Backplane, J2 RC6802_UI_Port, J3 BARREL_JACK, J4 DECODED, M1 Mounting, M2 Mounting, M3 Mounting, M4 Mounting, SW1 SST, SW2 RESET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

Commit message: CPU board layout done
Parts:
- removed SW1: SST, symbol SW_SPDT
- removed SW2: RESET, symbol SW_SPST
- added C7, C8: 100nF, Capacitors_THT:C_Disc_D4.7mm_W2.5mm_P5.00mm, symbol C
- added D1: HALT, LEDs:LED_D5.0mm, symbol LED_Small
- added D2: RESET, LEDs:LED_D5.0mm, symbol LED_Small
- added D3: NMI, LEDs:LED_D5.0mm, symbol LED_Small
- added D4: IRQ, LEDs:LED_D5.0mm, symbol LED_Small
- added D5: I/O, LEDs:LED_D5.0mm, symbol LED_Small
- added D6: R/W, LEDs:LED_D5.0mm, symbol LED_Small
- added D7: VMA, LEDs:LED_D5.0mm, symbol LED_Small
- added D8: E, LEDs:LED_D5.0mm, symbol LED_Small
- added JP3: LED_EN, Pin_Headers:Pin_Header_Straight_1x03_Pitch2.54mm, symbol Jumper_NC_Dual
- added R10, R11, R12, R5, R6, R7, R8, R9: 220, Resistors_THT:R_Axial_DIN0207_L6.3mm_D2.5mm_P7.62mm_Horizontal, symbol R
- added R4: 3k3, Resistors_THT:R_Axial_DIN0207_L6.3mm_D2.5mm_P10.16mm_Horizontal, symbol R
- added unit 6 of U4
- added U7: 74LS138, Housings_DIP:DIP-16_W7.62mm_Socket, symbol 74LS138
- added U8: 74LS240, Housings_DIP:DIP-20_W7.62mm_Socket, symbol 74LS240
- C11: renamed from C8; footprint (none) -> Capacitors_THT:C_Disc_D4.7mm_W2.5mm_P5.00mm
- C9: footprint (none) -> Capacitors_THT:C_Disc_D4.7mm_W2.5mm_P5.00mm
- J1: footprint (none) -> Pin_Headers:Pin_Header_Angled_1x39_Pitch2.54mm
- J2: footprint (none) -> Pin_Headers:Pin_Header_Straight_2x20_Pitch2.54mm
- J4, JP1: footprint (none) -> Pin_Headers:Pin_Header_Straight_1x03_Pitch2.54mm
- JP2: value EX_RAM_CS -> RAM_SEL; footprint (none) -> Pin_Headers:Pin_Header_Straight_1x03_Pitch2.54mm
- R1, R2, R3: value 10k -> 3k3; footprint (none) -> Resistors_THT:R_Axial_DIN0207_L6.3mm_D2.5mm_P10.16mm_Horizontal
- U1, U6: footprint (none) -> Housings_DIP:DIP-40_W15.24mm_Socket
- U4: footprint (none) -> Housings_DIP:DIP-14_W7.62mm_Socket
- Y1: footprint (none) -> Crystals:Crystal_HC49-U_Vertical
- renumbered C7 to C10
Connections:
- net labels added: IO0, IO1, IO2, IO3, IO4, IO5, IO6, IO7, ~SST
- wire segments 279 -> 332
- no-connect marks 35 -> 17
Other:
- note added: "$E000"
- note added: "RC6802 Microchicken computer as explained in the book "22 Micro-computer projects:\nTo build, use and learn" by Daniel Metzger. Hardware changed slightly to add a\nsecondary 74LS138 to further divide device area ($2000-$3FFF), original addresses used\nin code examples should be unchanged from original memory map."
- note removed: "$F000"
- moved on the sheet: C1, C2, C3, C4, C5, C6, R1, R2, R3
