File: RC6802 CPU/RC6802 CPU.kicad_pcb (KiCad board)
At the start: 2 copper layers, 99.1 x 99.1 mm, 53 parts, among them J1 RC6802_Backplane, J2 RC6802_UI_Port, J3 BARREL_JACK, J4 DECODED, M1 Mounting, M2 Mounting, M3 Mounting, M4 Mounting, U1 MC6802, U2 HM62256BLP-7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

Commit message: Updated software
Changed lines of the file:
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@@
       (effects (font (size 1 1) (thickness 0.15)))
     )
-    (fp_text value 3k3 (at 6.985 0) (layer F.SilkS)
+    (fp_text value 3k3 (at 6.35 0) (layer F.SilkS)
       (effects (font (size 1 1) (thickness 0.15)))
     )
@@
     (descr "Resistor, Axial_DIN0207 series, Axial, Horizontal, pin pitch=10.16mm, 0.25W = 1/4W, length*diameter=6.3*2.5mm^2, http://cdn-reichelt.de/documents/datenblatt/B400/1_4W%23YAG.pdf")
     (tags "Resistor Axial_DIN0207 series Axial Horizontal pin pitch 10.16mm 0.25W = 1/4W length 6.3mm diameter 2.5mm")
-    (fp_text reference R3 (at 6.985 0 90) (layer F.SilkS)
+    (fp_text reference R3 (at 3.175 0 90) (layer F.SilkS)
       (effects (font (size 1 1) (thickness 0.15)))
     )
-    (fp_text value 3k3 (at 3.81 0) (layer F.SilkS)
+    (fp_text value 3k3 (at 6.35 0) (layer F.SilkS)
       (effects (font (size 1 1) (thickness 0.15)))
     )

Commit message: Error in MC6802 footprint
Connections:
- U1 pad 37: (no net) -> /E
- U1 pad 7: /E -> (no net)
Routing:
- net /E: track 191.6 -> 196.7 mm
Changed lines of the file:
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@@
     (links 263)
     (no_connects 0)
-    (area 93.345 43.815 204.470001 161.290001)
+    (area 100.254999 48.184999 199.465001 147.395001)
     (thickness 1.6)
     (drawings 125)
-    (tracks 2073)
+    (tracks 2074)
     (zones 0)
     (modules 53)
@@
     (pad 26 thru_hole oval (at 15.24 35.56) (size 1.6 1.6) (drill 0.8) (layers *.Cu *.Mask)
       (net 28 /D7))
-    (pad 7 thru_hole oval (at 0 15.24) (size 1.6 1.6) (drill 0.8) (layers *.Cu *.Mask)
-      (net 47 /E))
+    (pad 7 thru_hole oval (at 0 15.24) (size 1.6 1.6) (drill 0.8) (layers *.Cu *.Mask))
     (pad 27 thru_hole oval (at 15.24 33.02) (size 1.6 1.6) (drill 0.8) (layers *.Cu *.Mask)
       (net 27 /D6))
@@
     (pad 17 thru_hole oval (at 0 40.64) (size 1.6 1.6) (drill 0.8) (layers *.Cu *.Mask)
       (net 10 /A8))
-    (pad 37 thru_hole oval (at 15.24 7.62) (size 1.6 1.6) (drill 0.8) (layers *.Cu *.Mask))
+    (pad 37 thru_hole oval (at 15.24 7.62) (size 1.6 1.6) (drill 0.8) (layers *.Cu *.Mask)
+      (net 47 /E))
     (pad 18 thru_hole oval (at 0 43.18) (size 1.6 1.6) (drill 0.8) (layers *.Cu *.Mask)
       (net 9 /A9))
@@
   (segment (start 182.88 83.82) (end 194.945 83.82) (width 0.25) (layer F.Cu) (net 46))
   (segment (start 195.58 120.015) (end 195.58 120.65) (width 0.25) (layer F.Cu) (net 46))
+  (segment (start 142.24 98.425) (end 142.24 90.805) (width 0.25) (layer B.Cu) (net 47))
+  (segment (start 142.24 123.825) (end 142.24 98.425) (width 0.25) (layer B.Cu) (net 47))
+  (segment (start 152.4 91.44) (end 142.875 91.44) (width 0.25) (layer F.Cu) (net 47))
+  (via (at 142.24 90.805) (size 0.6) (drill 0.4) (layers F.Cu B.Cu) (net 47))
+  (segment (start 142.875 91.44) (end 142.24 90.805) (width 0.25) (layer F.Cu) (net 47))
   (segment (start 148.59 81.28) (end 150.495 81.28) (width 0.25) (layer B.Cu) (net 47))
   (segment (start 149.225 57.785) (end 149.86 58.42) (width 0.25) (layer F.Cu) (net 47))
@@
   (segment (start 147.955 80.645) (end 148.59 81.28) (width 0.25) (layer B.Cu) (net 47))
   (segment (start 142.24 83.185) (end 142.24 81.28) (width 0.25) (layer B.Cu) (net 47))
-  (segment (start 142.24 98.425) (end 142.24 83.185) (width 0.25) (layer B.Cu) (net 47))
+  (segment (start 142.24 90.805) (end 142.24 83.185) (width 0.25) (layer B.Cu) (net 47))
   (segment (start 116.205 128.27) (end 116.84 128.27) (width 0.25) (layer F.Cu) (net 47))
   (segment (start 104.775 127) (end 106.045 128.27) (width 0.25) (layer F.Cu) (net 47))
@@
   (via (at 117.475 127.635) (size 0.6) (drill 0.4) (layers F.Cu B.Cu) (net 47))
   (segment (start 116.84 128.27) (end 117.475 127.635) (width 0.25) (layer F.Cu) (net 47))
-  (segment (start 137.16 99.06) (end 141.605 99.06) (width 0.25) (layer F.Cu) (net 47))
-  (via (at 142.24 98.425) (size 0.6) (drill 0.4) (layers F.Cu B.Cu) (net 47))
-  (segment (start 141.605 99.06) (end 142.24 98.425) (width 0.25) (layer F.Cu) (net 47))
-  (segment (start 142.24 123.825) (end 142.24 98.425) (width 0.25) (layer B.Cu) (net 47))
   (segment (start 135.89 123.19) (end 141.605 123.19) (width 0.25) (layer F.Cu) (net 47))
   (segment (start 130.81 123.19) (end 135.89 123.19) (width 0.25) (layer F.Cu) (net 47))

Commit message: Fixed CPU bugs
Parts:
- C11, C9: value 33pF -> 22pF
Other:
- board text added: "5v DC"
- board text added: "CPU Revision B"
- board text removed: "CPU Revision A"
Changed lines of the file:
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@@
     (area 100.254999 48.184999 199.465001 147.395001)
     (thickness 1.6)
-    (drawings 125)
+    (drawings 134)
     (tracks 2074)
     (zones 0)
@@
       (effects (font (size 1 1) (thickness 0.15)))
     )
-    (fp_text value 33pF (at 2.54 0 180) (layer B.SilkS)
+    (fp_text value 22pF (at 2.54 0 180) (layer B.SilkS)
       (effects (font (size 1 1) (thickness 0.15)) (justify mirror))
     )
@@
       (effects (font (size 1 1) (thickness 0.15)))
     )
-    (fp_text value 33pF (at 2.54 0 270) (layer B.SilkS)
+    (fp_text value 22pF (at 2.54 0 270) (layer B.SilkS)
       (effects (font (size 1 1) (thickness 0.15)) (justify mirror))
     )
@@
     )
   )
+  (gr_text "5v DC" (at 107.315 57.15) (layer B.SilkS)
+    (effects (font (size 0.8 0.8) (thickness 0.1)) (justify mirror))
+  )
+  (gr_line (start 110.49 64.77) (end 110.49 62.23) (angle 90) (layer B.SilkS) (width 0.2))
+  (gr_line (start 109.22 64.77) (end 110.49 64.77) (angle 90) (layer B.SilkS) (width 0.2))
+  (gr_line (start 104.14 64.77) (end 105.41 64.77) (angle 90) (layer B.SilkS) (width 0.2))
+  (gr_line (start 104.14 62.23) (end 104.14 64.77) (angle 90) (layer B.SilkS) (width 0.2))
+  (gr_line (start 110.49 56.515) (end 110.49 58.42) (angle 90) (layer B.SilkS) (width 0.2))
+  (gr_line (start 104.14 55.88) (end 104.14 58.42) (angle 90) (layer B.SilkS) (width 0.2))
+  (gr_line (start 110.49 55.88) (end 104.14 55.88) (angle 90) (layer B.SilkS) (width 0.2))
+  (gr_line (start 110.49 56.515) (end 110.49 55.88) (angle 90) (layer B.SilkS) (width 0.2))
+  (gr_line (start 182.88 122.555) (end 185.42 122.555) (angle 90) (layer B.SilkS) (width 0.2))
+  (gr_line (start 182.88 121.285) (end 182.88 122.555) (angle 90) (layer B.SilkS) (width 0.2))
+  (gr_line (start 193.04 122.555) (end 193.04 121.285) (angle 90) (layer B.SilkS) (width 0.2))
+  (gr_line (start 195.58 122.555) (end 193.04 122.555) (angle 90) (layer B.SilkS) (width 0.2))
   (gr_text "On-Chip RAM" (at 144.78 93.98) (layer B.SilkS)
     (effects (font (size 1 1) (thickness 0.15)) (justify mirror))
@@
     (effects (font (size 0.8 0.8) (thickness 0.1)))
   )
-  (gr_line (start 187.96 122.555) (end 187.96 121.285) (angle 90) (layer B.SilkS) (width 0.2))
-  (gr_line (start 185.42 122.555) (end 187.96 122.555) (angle 90) (layer B.SilkS) (width 0.2))
   (gr_line (start 185.42 121.285) (end 185.42 122.555) (angle 90) (layer B.SilkS) (width 0.2))
   (gr_line (start 195.58 122.555) (end 195.58 121.285) (angle 90) (layer B.SilkS) (width 0.2))
-  (gr_line (start 195.58 122.555) (end 198.12 122.555) (angle 90) (layer B.SilkS) (width 0.2))
-  (gr_line (start 198.12 121.285) (end 198.12 122.555) (angle 90) (layer B.SilkS) (width 0.2))
   (gr_text github.com/tebl (at 184.15 132.08) (layer F.SilkS)
     (effects (font (size 1 1) (thickness 0.15)))
   )
-  (gr_text "CPU Revision A" (at 184.785 130.175) (layer F.SilkS)
+  (gr_text "CPU Revision B" (at 184.785 130.175) (layer F.SilkS)
     (effects (font (size 1 1) (thickness 0.15)))
   )
