File: RC6802 Serial Chicken/RC6802 Serial Chicken.sch (KiCad schematic (older format))
At the start: 17 parts, among them J1 RC6802_Backplane, J2 FTDI, J3 ADDRESS, U1 MC6850, U2 74LS04, U3 74LS138, X1 1.8432Mhz

Commit message: Updated software
Parts:
- J2: footprint (none) -> Pin_Headers:Pin_Header_Angled_1x06_Pitch2.54mm
- J3: footprint (none) -> Pin_Headers:Pin_Header_Straight_2x07_Pitch2.54mm
- JP1, JP2: footprint (none) -> Pin_Headers:Pin_Header_Straight_1x02_Pitch2.54mm
- JP3: footprint (none) -> Pin_Headers:Pin_Header_Straight_1x03_Pitch2.54mm
- JP4: renamed from JP?; footprint (none) -> Pin_Headers:Pin_Header_Straight_1x03_Pitch2.54mm
- R1, R2, R3: footprint (none) -> Resistors_THT:R_Axial_DIN0207_L6.3mm_D2.5mm_P10.16mm_Horizontal
- U1: footprint (none) -> Housings_DIP:DIP-24_W15.24mm_Socket
- U2: footprint (none) -> Housings_DIP:DIP-14_W7.62mm_Socket
Connections:
- net ~IRQ: now also J1.22 (IRQ)
- no-connect marks 27 -> 26
Changed lines of the file:
@@
 F 0 "U1" H 2350 5450 60  0000 C CNN
 F 1 "MC6850" V 2775 4500 60  0000 C CNN
-F 2 "" H 2775 4100 60  0000 C CNN
+F 2 "Housings_DIP:DIP-24_W15.24mm_Socket" H 2775 4100 60  0001 C CNN
 F 3 "" H 2775 4100 60  0000 C CNN
 	1    2775 4750
@@
 F 0 "J3" H 10775 3300 50  0000 C CNN
 F 1 "ADDRESS" H 10775 2500 50  0000 C CNN
-F 2 "" H 10725 2900 50  0001 C CNN
+F 2 "Pin_Headers:Pin_Header_Straight_2x07_Pitch2.54mm" H 10725 2900 50  0001 C CNN
 F 3 "" H 10725 2900 50  0001 C CNN
 	1    10725 2900
@@
 F 0 "JP3" H 10400 3850 50  0000 L CNN
 F 1 "CLOCK_SEL" H 10350 4050 50  0000 C BNN
-F 2 "" H 10350 3950 50  0001 C CNN
+F 2 "Pin_Headers:Pin_Header_Straight_1x03_Pitch2.54mm" H 10350 3950 50  0001 C CNN
 F 3 "" H 10350 3950 50  0001 C CNN
 	1    10350 3950
@@
 F 0 "J2" H 6250 4600 50  0000 C CNN
 F 1 "FTDI" H 6250 3900 50  0000 C CNN
-F 2 "" H 6250 4300 50  0001 C CNN
+F 2 "Pin_Headers:Pin_Header_Angled_1x06_Pitch2.54mm" H 6250 4300 50  0001 C CNN
 F 3 "" H 6250 4300 50  0001 C CNN
 	1    6250 4300
@@
 F 0 "R2" V 4525 4200 50  0000 C CNN
 F 1 "2k7" V 4625 4200 50  0000 C CNN
-F 2 "" V 4555 4200 50  0001 C CNN
+F 2 "Resistors_THT:R_Axial_DIN0207_L6.3mm_D2.5mm_P10.16mm_Horizontal" V 4555 4200 50  0001 C CNN
 F 3 "" H 4625 4200 50  0001 C CNN
 	1    4625 4200
@@
 F 0 "R3" V 4725 4300 50  0000 C CNN
 F 1 "2k7" V 4625 4300 50  0000 C CNN
-F 2 "" V 4555 4300 50  0001 C CNN
+F 2 "Resistors_THT:R_Axial_DIN0207_L6.3mm_D2.5mm_P10.16mm_Horizontal" V 4555 4300 50  0001 C CNN
 F 3 "" H 4625 4300 50  0001 C CNN
 	1    4625 4300
@@
 F 0 "U2" H 2445 10490 50  0000 C CNN
 F 1 "74LS04" H 2440 10250 50  0000 C CNN
-F 2 "" H 2250 10375 50  0001 C CNN
+F 2 "Housings_DIP:DIP-14_W7.62mm_Socket" H 2250 10375 50  0001 C CNN
 F 3 "" H 2250 10375 50  0001 C CNN
 	1    2250 10375
@@
 F 0 "U2" H 2770 10490 50  0000 C CNN
 F 1 "74LS04" H 2765 10250 50  0000 C CNN
-F 2 "" H 2575 10375 50  0001 C CNN
+F 2 "Housings_DIP:DIP-14_W7.62mm_Socket" H 2575 10375 50  0001 C CNN
 F 3 "" H 2575 10375 50  0001 C CNN
 	2    2575 10375
@@
 F 0 "U2" H 3095 10490 50  0000 C CNN
 F 1 "74LS04" H 3090 10250 50  0000 C CNN
-F 2 "" H 2900 10375 50  0001 C CNN
+F 2 "Housings_DIP:DIP-14_W7.62mm_Socket" H 2900 10375 50  0001 C CNN
 F 3 "" H 2900 10375 50  0001 C CNN
 	3    2900 10375
@@
 F 0 "U2" H 3420 10490 50  0000 C CNN
 F 1 "74LS04" H 3415 10250 50  0000 C CNN
-F 2 "" H 3225 10375 50  0001 C CNN
+F 2 "Housings_DIP:DIP-14_W7.62mm_Socket" H 3225 10375 50  0001 C CNN
 F 3 "" H 3225 10375 50  0001 C CNN
 	4    3225 10375
@@
 F 0 "U2" H 3745 10490 50  0000 C CNN
 F 1 "74LS04" H 3740 10250 50  0000 C CNN
-F 2 "" H 3550 10375 50  0001 C CNN
+F 2 "Housings_DIP:DIP-14_W7.62mm_Socket" H 3550 10375 50  0001 C CNN
 F 3 "" H 3550 10375 50  0001 C CNN
 	5    3550 10375
@@
 F 0 "U2" H 4920 3140 50  0000 C CNN
 F 1 "74LS04" H 4915 2900 50  0000 C CNN
-F 2 "" H 4725 3025 50  0001 C CNN
+F 2 "Housings_DIP:DIP-14_W7.62mm_Socket" H 4725 3025 50  0001 C CNN
 F 3 "" H 4725 3025 50  0001 C CNN
 	6    4725 3025
@@
 F 0 "R1" V 4050 2800 50  0000 C CNN
 F 1 "2k2" V 4150 2800 50  0000 C CNN
-F 2 "" V 4080 2800 50  0001 C CNN
+F 2 "Resistors_THT:R_Axial_DIN0207_L6.3mm_D2.5mm_P10.16mm_Horizontal" V 4080 2800 50  0001 C CNN
 F 3 "" H 4150 2800 50  0001 C CNN
 	1    4150 2800
@@
 F 0 "JP1" H 5350 3105 50  0000 C CNN
 F 1 "RTS_EN" H 5360 2965 50  0000 C CNN
-F 2 "" H 5350 3025 50  0001 C CNN
+F 2 "Pin_Headers:Pin_Header_Straight_1x02_Pitch2.54mm" H 5350 3025 50  0001 C CNN
 F 3 "" H 5350 3025 50  0001 C CNN
 	1    5350 3025
@@
 F 0 "JP2" H 5350 3930 50  0000 C CNN
 F 1 "USB_PWR" H 5360 3790 50  0000 C CNN
-F 2 "" H 5350 3850 50  0001 C CNN
+F 2 "Pin_Headers:Pin_Header_Straight_1x02_Pitch2.54mm" H 5350 3850 50  0001 C CNN
 F 3 "" H 5350 3850 50  0001 C CNN
 	1    5350 3850
@@
 NoConn ~ 14925 7125
 NoConn ~ 14925 7325
-NoConn ~ 14925 7425
 NoConn ~ 14925 7625
 NoConn ~ 14925 8125
@@
 A0
 $Comp
-L Jumper_NC_Dual JP?
+L Jumper_NC_Dual JP4
 U 1 1 5D890577
 P 3675 3025
-F 0 "JP?" H 3775 2900 50  0000 L CNN
+F 0 "JP4" H 3775 2900 50  0000 L CNN
 F 1 "IRQ_OUT_SEL" H 3675 3125 50  0000 C BNN
-F 2 "" H 3675 3025 50  0001 C CNN
+F 2 "Pin_Headers:Pin_Header_Straight_1x03_Pitch2.54mm" H 3675 3025 50  0001 C CNN
 F 3 "" H 3675 3025 50  0001 C CNN
 	1    3675 3025
@@
 Text Notes 5875 4600 0    60   ~ 0
 GND
+Wire Wire Line
+	14925 7425 14525 7425
+Entry Wire Line
+	14525 7425 14425 7325
+Text Label 14900 7425 2    60   ~ 0
+~IRQ
 $EndSCHEMATC
